File: 2023/SAL FP/keyboard/SAL-FP_Keyboard-LogicBoard/SAL-FP_Keyboard-LogicBoard.kicad_sch (KiCad schematic)
At the start: 11 parts, among them J1 Conn_01x12_Pin, J2 Conn_01x12_Pin, J3 Conn_01x12_Pin, Q2 Q_NPN_EBC, SW1 SW_Push

Commit message: update 2023-10-12
Parts:
- renumbered Q2 to Q1
Connections:
- net RX renamed D2
- net SCL renamed D0
- net SDA renamed D1
- net TX renamed D3
Changed lines of the file:
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@@
     (effects (font (size 1.27 1.27)) (justify right bottom))
   )
-  (label "TX" (at 147.32 91.44 0) (fields_autoplaced)
+  (label "D3" (at 147.32 91.44 0) (fields_autoplaced)
     (effects (font (size 1.27 1.27)) (justify left bottom))
   )
@@
     (effects (font (size 1.27 1.27)) (justify left bottom))
   )
-  (label "SDA" (at 147.32 101.6 0) (fields_autoplaced)
+  (label "D1" (at 147.32 101.6 0) (fields_autoplaced)
     (effects (font (size 1.27 1.27)) (justify left bottom))
   )
@@
     (effects (font (size 1.27 1.27)) (justify left bottom))
   )
-  (label "SCL" (at 147.32 104.14 0) (fields_autoplaced)
+  (label "D0" (at 147.32 104.14 0) (fields_autoplaced)
     (effects (font (size 1.27 1.27)) (justify left bottom))
   )
@@
     (effects (font (size 1.27 1.27)) (justify left bottom))
   )
-  (label "RX" (at 147.32 93.98 0) (fields_autoplaced)
+  (label "D2" (at 147.32 93.98 0) (fields_autoplaced)
     (effects (font (size 1.27 1.27)) (justify left bottom))
   )
@@
   (symbol (lib_id "Device:Q_NPN_EBC") (at 160.02 127 0) (unit 1)
     (in_bom yes) (on_board yes) (dnp no) (fields_autoplaced)
-    (property "Reference" "Q2" (at 165.1 125.73 0)
+    (property "Reference" "Q1" (at 165.1 125.73 0)
       (effects (font (size 1.27 1.27)) (justify left))
     )
@@
       (project "SAL-FP_Keyboard-LogicBoard"
         (path "/72a17f24-2f8a-4922-9ca3-2a63e0a6b754"
-          (reference "Q2") (unit 1)
-        )
-      )
+          (reference "Q1") (unit 1)
+        )
+      )
