File: 2023/SAL FP/keyboard/SAL-FP_Keyboard-LogicBoard/SAL-FP_Keyboard-LogicBoard.kicad_pcb (KiCad board)
At the start: 2 copper layers, 47 x 30 mm, 11 parts, among them J1 Conn_01x12_Pin, J2 Conn_01x12_Pin, J3 Conn_01x12_Pin, Q2 Q_NPN_EBC, SW1 SW_Push

Commit message: update 2023-10-12
Parts:
- removed Q2: Q_NPN_EBC, Package_TO_SOT_THT:TO-92
- added Q1: Q_NPN_EBC, Package_TO_SOT_THT:TO-92, F.Cu at (144.1, 109.2)
- moved SW1 7.91 mm to (145.8, 116.1), turned to -90 degrees
Connections:
- net /RX renamed /D2
- net /SCL renamed /D0
- net /SDA renamed /D1
- net /TX renamed /D3
Routing:
- net /RST: track 33.3 -> 28.8 mm
Other:
- board size 47 x 30 mm -> 44.5 x 30 mm
