File: 2023/SAL FP/keyboard/SAL-FP_Keyboard.kicad_pcb (KiCad board)
At the start: 2 copper layers, 108 x 31.3 mm, 8 parts, among them J1 Conn_01x04_Pin, J2 Conn_01x12_Socket, J3 Conn_01x12_Socket, SW1 SW_Push_LED, SW2 SW_Push_LED, SW3 SW_Push_LED, SW4 SW_Push_LED, SW5 SW_Push_LED

Commit message: Adding a week of random stuff.
Other:
- outline, holes or cut-outs redrawn
Changed lines of the file:
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@@
     (pad_to_mask_clearance 0)
     (aux_axis_origin 146.71 120.89)
-    (grid_origin 92.71 135.89)
+    (grid_origin 54.61 135.89)
     (pcbplotparams
       (layerselection 0x00010fc_ffffffff)
@@
       (viasonmask false)
       (mode 1)
-      (useauxorigin false)
+      (useauxorigin true)
       (hpglpennumber 1)
       (hpglpenspeed 20)
@@
       (outputformat 1)
       (mirror false)
-      (drillshape 1)
+      (drillshape 0)
       (scaleselection 1)
-      (outputdirectory "")
+      (outputdirectory "fab/")
     )
   )
@@
     )
   )
+  (gr_circle (center 54.61 135.89) (end 56.61 135.89)
+    (stroke (width 0.1) (type default)) (fill none) (layer "Edge.Cuts"))
+  (gr_circle (center 130.81 135.89) (end 132.81 135.89)
+    (stroke (width 0.1) (type default)) (fill none) (layer "Edge.Cuts"))
+  (gr_circle (center 92.71 135.89) (end 94.71 135.89)
+    (stroke (width 0.1) (type default)) (fill none) (layer "Edge.Cuts"))
   (gr_rect (start 38.71 120.89) (end 146.71 152.16)
     (stroke (width 0.1) (type default)) (fill none) (layer "Edge.Cuts"))
+  (gr_circle (center 73.66 135.89) (end 75.66 135.89)
+    (stroke (width 0.1) (type default)) (fill none) (layer "Edge.Cuts"))
+  (gr_circle (center 111.76 135.89) (end 113.76 135.89)
+    (stroke (width 0.1) (type default)) (fill none) (layer "Edge.Cuts"))
   (segment (start 102.108 132.842) (end 103.124 132.842) (width 0.45) (layer "B.Cu") (net 1))
