File: 2023/SAL FP/keyboard/SAL-FP_Keyboard-LogicBoard-Modbus/SAL-FP_Keyboard-LogicBoard.kicad_sch (KiCad schematic)
At the start: 13 parts, among them J1 Conn_01x12_Pin, J2 Conn_01x12_Pin, J3 Conn_01x12_Pin, J5 RS485, U1 MCP1700x-330xxMB, U2 MAX3485, U3 EFM8BB10F8G-A-SOIC16

Commit message: Adding a week of random stuff.
Other:
- note added: "Current Limiting Resistors Needed!"
Changed lines of the file:
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@@
     (effects (font (size 1.27 1.27)) (justify left bottom))
+  )
+  (text "Current Limiting Resistors Needed!" (at 168.91 77.47 0)
+    (effects (font (size 2.54 2.54)) (justify left bottom))
   )
   (label "LED1" (at 229.87 40.64 0) (fields_autoplaced)
