File: 2023/SAL FP/power_distribution_board/power_distribution_board.kicad_sch (KiCad schematic)
At the start: 13 parts, among them J1 hal, J2 daisy, J3 web, J4 switch, J5 axxs, J6 -, J7 +, J8 acc, J9 audio, U1 MINI-360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

Commit message: weekend work.
Connections:
- net GND: now also J1.1 (Pin_1), J2.1 (Pin_1), J3.1 (Pin_1), J9.1 (Pin_1), U1.3 (out-), U2.3 (out-), U3.3 (out-), U4.3 (out-)
Changed lines of the file:
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@@
 (kicad_sch (version 20230121) (generator eeschema)
   (paper "A4")
+  (junction (at 63.5 76.2) (diameter 0) (color 0 0 0 0)
+  )
+  (junction (at 149.86 76.2) (diameter 0) (color 0 0 0 0)
+  )
+  (junction (at 106.68 76.2) (diameter 0) (color 0 0 0 0)
+  )
+  (junction (at 193.04 76.2) (diameter 0) (color 0 0 0 0)
+  )
   (wire (pts (xy 124.46 76.2) (xy 127 76.2))
     (stroke (width 0) (type default))
@@
     (stroke (width 0) (type default))
   )
+  (wire (pts (xy 63.5 76.2) (xy 63.5 78.74))
+    (stroke (width 0) (type default))
+  )
   (wire (pts (xy 31.75 29.21) (xy 31.75 31.75))
     (stroke (width 0) (type default))
@@
     (stroke (width 0) (type default))
   )
+  (wire (pts (xy 193.04 76.2) (xy 193.04 78.74))
+    (stroke (width 0) (type default))
+  )
   (wire (pts (xy 63.5 71.12) (xy 60.96 71.12))
     (stroke (width 0) (type default))
@@
   )
   (wire (pts (xy 60.96 76.2) (xy 63.5 76.2))
+    (stroke (width 0) (type default))
+  )
+  (wire (pts (xy 106.68 76.2) (xy 106.68 78.74))
+    (stroke (width 0) (type default))
+  )
+  (wire (pts (xy 149.86 76.2) (xy 149.86 78.74))
     (stroke (width 0) (type default))
   )
@@
     )
   )
+  (symbol (lib_id "power:GND") (at 63.5 78.74 0) (unit 1)
+    (in_bom yes) (on_board yes) (dnp no) (fields_autoplaced)
+    (property "Reference" "#PWR017" (at 63.5 85.09 0)
+      (effects (font (size 1.27 1.27)) hide)
+    )
+    (property "Value" "GND" (at 63.5 83.82 0)
+      (effects (font (size 1.27 1.27)))
+    )
+    (property "Footprint" "" (at 63.5 78.74 0)
+      (effects (font (size 1.27 1.27)) hide)
+    )
+    (property "Datasheet" "" (at 63.5 78.74 0)
+      (effects (font (size 1.27 1.27)) hide)
+    )
+    (pin "1")
+    (instances
+      (project "power_distribution_board"
+        (path "/3ebf3a73-04b6-4f83-b3c8-3031e5cfeb99"
+          (reference "#PWR017") (unit 1)
+        )
+      )
+    )
+  )
   (symbol (lib_id "power:+12V") (at 38.1 68.58 0) (unit 1)
     (in_bom yes) (on_board yes) (dnp no) (fields_autoplaced)
@@
         )
       )
+    )
+  )
+  (symbol (lib_id "power:GND") (at 149.86 78.74 0) (unit 1)
+    (in_bom yes) (on_board yes) (dnp no) (fields_autoplaced)
+    (property "Reference" "#PWR019" (at 149.86 85.09 0)
+      (effects (font (size 1.27 1.27)) hide)
+    )
+    (property "Value" "GND" (at 149.86 83.82 0)
+      (effects (font (size 1.27 1.27)))
+    )
+    (property "Footprint" "" (at 149.86 78.74 0)
+      (effects (font (size 1.27 1.27)) hide)
+    )
+    (property "Datasheet" "" (at 149.86 78.74 0)
+      (effects (font (size 1.27 1.27)) hide)
+    )
+    (pin "1")
+    (instances
+      (project "power_distribution_board"
+        (path "/3ebf3a73-04b6-4f83-b3c8-3031e5cfeb99"
+          (reference "#PWR019") (unit 1)
+        )
+      )
+    )
+  )
+  (symbol (lib_id "power:GND") (at 193.04 78.74 0) (unit 1)
+    (in_bom yes) (on_board yes) (dnp no) (fields_autoplaced)
+    (property "Reference" "#PWR020" (at 193.04 85.09 0)
+      (effects (font (size 1.27 1.27)) hide)
+    )
+    (property "Value" "GND" (at 193.04 83.82 0)
+      (effects (font (size 1.27 1.27)))
+    )
+    (property "Footprint" "" (at 193.04 78.74 0)
+      (effects (font (size 1.27 1.27)) hide)
+    )
+    (property "Datasheet" "" (at 193.04 78.74 0)
+      (effects (font (size 1.27 1.27)) hide)
+    )
+    (pin "1")
+    (instances
+      (project "power_distribution_board"
+        (path "/3ebf3a73-04b6-4f83-b3c8-3031e5cfeb99"
+          (reference "#PWR020") (unit 1)
+        )
+      )
+    )
+  )
+  (symbol (lib_id "power:GND") (at 106.68 78.74 0) (unit 1)
+    (in_bom yes) (on_board yes) (dnp no) (fields_autoplaced)
+    (property "Reference" "#PWR018" (at 106.68 85.09 0)
+      (effects (font (size 1.27 1.27)) hide)
+    )
+    (property "Value" "GND" (at 106.68 83.82 0)
+      (effects (font (size 1.27 1.27)))
+    )
+    (property "Footprint" "" (at 106.68 78.74 0)
+      (effects (font (size 1.27 1.27)) hide)
+    )
+    (property "Datasheet" "" (at 106.68 78.74 0)
+      (effects (font (size 1.27 1.27)) hide)
+    )
+    (pin "1")
+    (instances
+      (project "power_distribution_board"
+        (path "/3ebf3a73-04b6-4f83-b3c8-3031e5cfeb99"
+          (reference "#PWR018") (unit 1)
+        )
+      )

Commit message: added work.
Removed large audio files.
Parts:
- added C1: 47u, Capacitor_THT:CP_Radial_D7.5mm_P2.50mm, symbol Device:C_Polarized
- added C2, C3: 10u, Capacitor_SMD:C_1206_3216Metric, symbol Device:C
Connections:
- net +12V: now also C1.1, C2.1, C3.1
- net GND: now also C1.2, C2.2, C3.2
Other:
- moved on the sheet: J6, J7
