File: 2026/autodir_sch/autodir_sch.kicad_sch (KiCad schematic)
At the start: 11 parts, among them J1 UART, J2 MB, J3 PROG, U1 CH32V003JxMx, U2 ST485E

Commit message: RS485 automatic direction schematic and reference PCB
Parts:
- C1, C2, C3: footprint Capacitor_SMD:C_0402_1005Metric -> Capacitor_SMD:C_0603_1608Metric
Connections:
- net A: now reaches J2.2 (Pin_2), R1.1, R2.2, U2.6 (A)
- net B: now reaches J2.3 (Pin_3), R1.2, R3.1, U2.7 (B)
Other:
- note added: "B A C"
Changed lines of the file:
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@@
 	(title_block
 		(title "RS485 Autodir")
-		(date "2026-01-30")
-		(rev "A0")
+		(date "2026-02-01")
+		(rev "A1")
 		(company "MAG Laboratory")
+	)
+	(text "B A C"
+		(exclude_from_sim no)
+		(at 199.39 93.218 0)
+		(effects
+			(font
+				(size 1.27 1.27)
+			)
+		)
 	)
 	(junction
@@
 		)
 	)
+	(label "A"
+		(at 194.31 74.93 0)
+		(effects
+			(font
+				(size 1.27 1.27)
+			)
+			(justify left bottom)
+		)
+	)
+	(label "B"
+		(at 194.31 80.01 0)
+		(effects
+			(font
+				(size 1.27 1.27)
+			)
+			(justify left bottom)
+		)
+	)
 	(symbol
 		(lib_id "Interface_UART:ST485E")
@@
 			)
 		)
-		(property "Footprint" "Capacitor_SMD:C_0402_1005Metric"
+		(property "Footprint" "Capacitor_SMD:C_0603_1608Metric"
 			(at 138.43 96.52 0)
 			(effects
@@
 			)
 		)
-		(property "Footprint" "Capacitor_SMD:C_0402_1005Metric"
+		(property "Footprint" "Capacitor_SMD:C_0603_1608Metric"
 			(at 129.54 96.52 0)
 			(effects
@@
 			)
 		)
-		(property "Footprint" "Capacitor_SMD:C_0402_1005Metric"
+		(property "Footprint" "Capacitor_SMD:C_0603_1608Metric"
 			(at 147.32 96.52 0)
 			(effects
