File: 2026/inverter_board/inverter_board.kicad_pcb (KiCad board)
At the start: 2 copper layers, 42.5 x 38.5 mm, 36 parts, among them J1 RJ12, J2 RJ12, J3 Modbus, J4 PROG, U1 CH32V003JxMx, U2 HCPL-0611, U3 HCPL-0611, U4 HCPL-0611, U5 MAX485E, U6 ME6209A50M3G

Commit message: Updated inverter decoder board to use a buck converter
Parts:
- removed U6: ME6209A50M3G, Package_TO_SOT_SMD:SOT-23
- added C15: 102, Capacitor_SMD:C_0603_1608Metric, F.Cu at (110.5, 146.0)
- added C16: 104, Capacitor_SMD:C_0603_1608Metric, B.Cu at (115.0, 152.9)
- added C17: 330, Capacitor_SMD:C_0603_1608Metric, F.Cu at (116.8, 155.4)
- added D1: SS210, Diode_SMD:D_SMA, B.Cu at (112.5, 151.2)
- added L1: 4.7u, Inductor_SMD:L_APV_APH0420, B.Cu at (118.3, 153.0)
- added R11: 2k, Resistor_SMD:R_0603_1608Metric, F.Cu at (110.5, 144.5)
- added R12: 124k, Resistor_SMD:R_0603_1608Metric, F.Cu at (116.8, 153.8)
- added R13: 23.7k, Resistor_SMD:R_0603_1608Metric, F.Cu at (116.8, 152.2)
- added U7: MD8941, Package_TO_SOT_SMD:SOT-23-6, F.Cu at (113.5, 153.6)
- C2: value 104 -> 106; footprint Capacitor_SMD:C_0603_1608Metric -> Capacitor_SMD:C_1206_3216Metric
- moved J4 4.11 mm to (110.5, 148.2)
- moved C14 3.52 mm to (103.5, 152.5), turned to 180 degrees
- moved R5 3.48 mm to (113.7, 141.0), turned to 180 degrees
- moved R10 3.07 mm to (106.0, 152.0), turned to -90 degrees
- moved C12 2.04 mm to (110.5, 153.5)
- moved C11 2.00 mm to (108.0, 153.9)
Connections:
- R5 pad 1: +5VP -> /UART
- R5 pad 2: Net-(U2-A) -> Net-(U2-C)
- U1 pad 6: /INV_DATA -> Net-(U1-PC2)
- U2 pad 2: Net-(U2-A) -> +5VP
- U2 pad 3: /UART -> Net-(U2-C)
Routing:
- net +5VP: track 76.8 -> 88.3 mm, vias 12 -> 16
- net Net-(U7-FB): track 0.00 -> 7.50 mm
- net Net-(D1-K): track 0.00 -> 7.35 mm, vias 0 -> 2
- net GNDPWR: track 125.7 -> 119.3 mm
- net /UART: track 30.2 -> 26.5 mm
- net Net-(U1-PC2): track 0.00 -> 3.69 mm
- net +12V: track 27.7 -> 25.0 mm
- net Net-(U2-C): track 0.00 -> 2.60 mm
- net Net-(U2-A): track 2.44 -> 0.00 mm
- net Net-(U7-BST): track 0.00 -> 2.34 mm, vias 0 -> 1
- net /INV_DATA: track 27.6 -> 26.1 mm
- net Net-(J4-Pin_2): track 3.36 -> 1.96 mm
- net /12V_FILT: track 9.78 -> 11.1 mm
- added copper zone on B.Cu, net Net-(D1-K)

Commit message: Refined inverter board's switching power supply
Routing:
- net GND: track 63.0 -> 64.2 mm, vias 3 -> 9
- net GNDPWR: vias 4 -> 12
- net +5VP: vias 16 -> 19
